File: Electronics/CNP_PCB/SwitchLogic.kicad_sch (KiCad schematic)
At the start: 7 parts, among them U2 74HC4051, U4 74HC4051, U5 SN74LVC1G3157DBVR

Commit message: changes made to button read logic
Parts:
- renumbered C4 to C?, R3 to R?, U2 to U?, U5 to U?
Connections:
- net KO7: no longer names the net of U?.4 (A7)
- no-connect marks 2 -> 4
Other:
- note added: "K0x → S2A S1A S0A KIx → S2B S1B S0B ----------------------------- K00 0 0 0 KI0 0 0 0 K01 0 0 1 KI1 0 0 1 K02 0 1 0 KI2 0 1 0 K03 0 1 1 KI3 0 1 1 K04 1 0 0 KI4 1 0 0 K05 1 0 1 KI5 1 0 1 K06 1 1 0 KI6 1 1 0 KI7 1 1 1"
- moved on the sheet: C5, C?, R10, R?, U4, U?
